Commit message: fix: preserve Go2 UTLiDAR frame and remove XT lidar

File: go2_description/urdf/go2_description.urdf (robot description, URDF)
Before this commit: robot go2_description, 48 links, 47 joints
Links:
- removed link Pandar64
- removed link PandarXT-32
- removed link hesai_lidar
- removed link pandar
- removed link rslidar
Joints:
- removed joint hesai_lidar_joint
- removed joint hesai_pandar64_joint
- removed joint hesai_pandar_joint
- removed joint hesai_pandar_xt_joint
- removed joint hesai_rslidar_joint
- joint utlidar_lidar_joint: origin xyz=0.28945 0 -0.046825 rpy=0 2.8782 0 -> xyz=0.3 0 -0.03 rpy=0.22 -3.00 2.05
